Commit message: gazebo unbreak

File: description/depth_camera.xacro (robot description, xacro)
@@ -1,9 +1,14 @@
 <?xml version="1.0"?>
-<robot xmlns:xacro="http://www.ros.org/wiki/xacro" >
+<robot xmlns:xacro="http://www.ros.org/wiki/xacro">
+    <!-- Include inertial macros -->
+    <xacro:include filename="inertial_macros.xacro"/>
+    <!-- Define colors -->
+  <!-- Joint connecting LiDAR to the chassis -->
     <joint name="camera_joint" type="fixed">
-        <parent link="chassis"/>
+        <parent link="chassis_link"/> <!-- Adjust parent link name as per your setup -->
         <child link="camera_link"/>
-        <origin xyz="0.305 0 0.08" rpy="0 0 0"/>
+        <origin xyz="0.18 0 0.215" rpy="0 0 0"/> <!-- Adjust origin and orientation if needed -->
     </joint>
+    <!-- Define the LiDAR link -->
     <link name="camera_link">
         <visual>
@@ -12,12 +17,15 @@
             </geometry>
             <material name="red"/>
+            <origin xyz="0 0 0" rpy="0 0 0"/> <!-- Adjust origin if needed -->
         </visual>
     </link>
-    <joint name="camera_optical_joint" type="fixed">
-        <parent link="camera_link"/>
-        <child link="camera_link_optical"/>
-        <origin xyz="0 0 0" rpy="${-pi/2} 0 ${-pi/2}"/>
+     <joint name="camera_optical_joint" type="fixed">
+        <parent link="chassis_link"/> <!-- Adjust parent link name as per your setup -->
+        <child link="camera_optical_link"/>
+        <origin xyz="0 0 0" rpy="${-pi/2} 0 ${-pi/2}"/> <!-- Adjust origin and orientation if needed -->
     </joint>
-    <link name="camera_link_optical"></link>
+     <link name="camera_optical_link">
+    </link>
+    <!-- Gazebo reference for LiDAR -->
     <gazebo reference="camera_link">
         <material>Gazebo/Red</material>
@@ -39,7 +47,7 @@
             </camera>
             <plugin name="camera_controller" filename="libgazebo_ros_camera.so">
-                <frame_name>camera_link_optical</frame_name>
+                <frame_name>camera_optical_link</frame_name>
                 <min_depth>0.1</min_depth>
-                <max_depth>100.0</max_depth>
+                <max_depth>100</max_depth>
             </plugin>
         </sensor>

File: description/robot.urdf.xacro (robot description, xacro)
@@ -11,5 +11,5 @@
     </xacro:unless>
     <xacro:include filename="lidar.xacro" />
-    <xacro:include filename="camera.xacro" />
-    <!-- <xacro:include filename="depth_camera.xacro" /> -->
+     <xacro:include filename="camera.xacro" />
+    <!-- <xacro:include filename="depth_camera.xacro" />  -->
 </robot>
