Commit message: robot final code

File: description/camera.xacro (robot description, xacro)
@@ -37,5 +37,5 @@
                 <horizontal_fov>1.089</horizontal_fov>
                 <image>
-                    <format>R8G8B8</format>
+                    <format>B8G8R8</format>
                     <width>640</width>
                     <height>480</height>
@@ -48,4 +48,6 @@
             <plugin name="camera_controller" filename="libgazebo_ros_camera.so">
                 <frame_name>camera_optical_link</frame_name>
+                <min_depth>0.1</min_depth>
+                <max_depth>100</max_depth>
             </plugin>
         </sensor>

File: description/robot_core.xacro (robot description, xacro)
@@ -73,5 +73,5 @@
     <visual>
       <geometry>
-        <cylinder radius="0.075" length="0.04"/>
+        <cylinder radius="0.056" length="0.04"/>
       </geometry>
       <material name="black"/>
@@ -79,5 +79,5 @@
     <collision>
       <geometry>
-        <cylinder radius="0.075" length="0.04"/>
+        <cylinder radius="0.056" length="0.04"/>
       </geometry>
     </collision>
@@ -103,5 +103,5 @@
     <visual>
       <geometry>
-        <cylinder radius="0.075" length="0.04"/>
+        <cylinder radius="0.056" length="0.04"/>
       </geometry>
       <material name="black"/>
@@ -109,5 +109,5 @@
     <collision>
       <geometry>
-        <cylinder radius="0.075" length="0.04"/>
+        <cylinder radius="0.056" length="0.04"/>
       </geometry>
     </collision>

File: description/ros2_control.xacro (robot description, xacro)
@@ -7,9 +7,9 @@
                 <param name="left_wheel_name">left_wheel_joint</param>
                 <param name="right_wheel_name">right_wheel_joint</param>
-                <param name="loop_rate">1</param>
-                <param name="device">/dev/ttyUSB0</param>
+                <param name="loop_rate">20</param>
+                <param name="device">/dev/serial/by-path/platform-fd500000.pcie-pci-0000:01:00.0-usb-0:1.1:1.0-port0</param>
                 <param name="baud_rate">57600</param>
                 <param name="timeout">1000</param>
-                <param name="enc_counts_per_rev">144</param>
+                <param name="enc_counts_per_rev">3030</param>
             </hardware>
             <joint name="left_wheel_joint">
